Commit message: feat(model): refresh URDF and meshes with CAD-derived inertias

File: urdf/model.urdf (robot description, URDF)
Before this commit: robot inverted_pendulum, 4 links, 3 joints
Links:
- removed link lid
- link arm: mass None -> 0.026; geometry visual mesh filename=package://meshes/arm.dae
- link base: geometry visual mesh filename=package://meshes/base.dae
- link pendulum: mass None -> 0.014
Joints:
- removed joint base_to_lid
- removed joint lid_to_arm
- added joint base_to_arm: type revolute, parent base, child arm, origin xyz=0 0 0.075 rpy=0 0 -1.57079, axis 0 0 1
