Commit message: fix(model): correct the URDF's pivot reach, visual meshes, and swing axis

File: urdf/model.urdf (robot description, URDF)
Before this commit: robot inverted_pendulum, 3 links, 2 joints
Links:
- added link lid; visual mesh filename=package://meshes/lid.stl scale=0.001 0.001 0.001
- link arm: geometry visual mesh filename=package://meshes/arm.stl scale=0.001 0.001 0.001
- link base: geometry visual mesh filename=package://meshes/base.stl scale=0.001 0.001 0.001
- link pendulum: geometry visual mesh filename=package://meshes/pendulum.stl scale=0.001 0.001 0.001
Joints:
- added joint base_to_lid: type fixed, parent base, child lid, origin xyz=0 0 0.070 rpy=0 0 0
- joint arm_to_pendulum: origin xyz=0 0 0.014 rpy=0 0 0 -> xyz=0.062 0 0.014 rpy=0 0 0
- joint base_to_arm: limit (none) -> lower=-2.35619449 upper=2.35619449 effort=0.4 velocity=196
